Commit message: updates and bug fixes

File: model/parametricArm.urdf (robot description, URDF)
Before this commit: robot parametric_arm, 5 links, 4 joints
Links:
- link link_0: geometry collision box size=0.05 0.05 1.5; visual box size=0.05 0.05 1.5
Joints:
- joint RY_1: origin xyz=0 0 -1.0 rpy=0 0 0 -> xyz=0 0 -1.5 rpy=0 0 0
