Commit message: final version

File: thrower/modified_model/parametricArm.urdf (robot description, URDF)
Before this commit: robot parametric_arm, 5 links, 4 joints
Links:
- link link_0: geometry collision box size=0.05 0.05 1; visual box size=0.05 0.05 1
- link link_1: geometry collision box size=0.05 0.05 1; visual box size=0.05 0.05 1
Joints:
- joint RY_1: origin xyz=0 0 -1.9957588556566768 rpy=0 0 0 -> xyz=0 0 -1 rpy=0 0 0
- joint arm_fixed_joint: origin xyz=0 0 -1.0361755480047945 rpy=0 0 0 -> xyz=0 0 -1 rpy=0 0 0

Commit message: fix tmp file bug

File: thrower/modified_model/parametricArm.urdf (robot description, URDF)
Before this commit: robot parametric_arm, 5 links, 4 joints
Links:
- link link_0: geometry collision box size=0.05 0.05 1.8882466653946577; visual box size=0.05 0.05 1.8882466653946577
- link link_1: geometry collision box size=0.05 0.05 1.0494091271408081; visual box size=0.05 0.05 1.0494091271408081
Joints:
- joint RY_1: origin xyz=0 0 -1 rpy=0 0 0 -> xyz=0 0 -1.8882466653946577 rpy=0 0 0
- joint arm_fixed_joint: origin xyz=0 0 -1 rpy=0 0 0 -> xyz=0 0 -1.0494091271408081 rpy=0 0 0
